Commit message: upgrade RGB camera to Kinect camera

File: src/my_robot/urdf/my_robot.xacro (robot description, xacro)
@@ -219,3 +219,10 @@
     <axis xyz="0 1 0" rpy="0 0 0"/>
   </joint>
+  <joint type="fixed" name="camera_optical_joint">
+    <origin xyz="0 0 0" rpy="-1.5707 0 -1.5707"/>
+    <parent link="camera_link"/>
+    <child link="camera_link_optical"/>
+  </joint>
+  <link name="camera_link_optical">
+  </link>
 </robot>

Commit message: change robot urdf file to fix camera_link name

File: src/my_robot/urdf/my_robot.xacro (robot description, xacro)
@@ -161,5 +161,5 @@
     <dynamics damping="1.0" friction="1.0"/>
   </joint>
-  <link name='camera'>
+  <link name='camera_link'>
     <inertial>
       <mass value=".1"/>
@@ -186,5 +186,5 @@
   <joint type="fixed" name="camera_joint">
     <origin xyz=".2 0 0" rpy="0 0 0"/>
-    <child link="camera"/>
+    <child link="camera_link"/>
     <parent link="chassis"/>
     <axis xyz="0 1 0" rpy="0 0 0"/>
